File: USB2CAN_TRA.sch (KiCad schematic (older format))
At the start: 24 parts

Commit message: Added labels to all components
Parts:
- gave numbers to parts that had none: 24
Changed lines of the file:
@@
 $EndDescr
 $Comp
-L MCU_ST_STM32F0:STM32F042C6Tx U?
+L MCU_ST_STM32F0:STM32F042C6Tx U4
 U 1 1 5E5656C2
 P 4350 3400
-AR Path="/5E564EEA/5E5656C2" Ref="U?"  Part="1"
+AR Path="/5E564EEA/5E5656C2" Ref="U4"  Part="1"
 AR Path="/5E45C906/5E5656C2" Ref="U?"  Part="1"
-F 0 "U?" H 4600 1900 50  0000 C CNN
+F 0 "U4" H 4600 1900 50  0000 C CNN
 F 1 "STM32F042C6Tx" H 4850 1800 50  0000 C CNN
 F 2 "Package_QFP:LQFP-48_7x7mm_P0.5mm" H 3850 2000 50  0001 R CNN
@@
 Connection ~ 4350 5100
 $Comp
-L Device:C C?
+L Device:C C29
 U 1 1 5E56F9CC
 P 6050 1050
-AR Path="/5E564EEA/5E56F9CC" Ref="C?"  Part="1"
+AR Path="/5E564EEA/5E56F9CC" Ref="C29"  Part="1"
 AR Path="/5E45C906/5E56F9CC" Ref="C?"  Part="1"
-F 0 "C?" H 6165 1096 50  0000 L CNN
+F 0 "C29" H 6165 1096 50  0000 L CNN
 F 1 "0.1u" H 6165 1005 50  0000 L CNN
 F 2 "" H 6088 900 50  0001 C CNN
@@
 	6050 850  6050 900
 $Comp
-L Device:C C?
+L Device:C C30
 U 1 1 5E570D68
 P 5150 1950
-AR Path="/5E564EEA/5E570D68" Ref="C?"  Part="1"
+AR Path="/5E564EEA/5E570D68" Ref="C30"  Part="1"
 AR Path="/5E45C906/5E570D68" Ref="C?"  Part="1"
-F 0 "C?" H 5265 1996 50  0000 L CNN
+F 0 "C30" H 5265 1996 50  0000 L CNN
 F 1 "0.1u" H 5265 1905 50  0000 L CNN
 F 2 "" H 5188 1800 50  0001 C CNN
@@
 $EndComp
 $Comp
-L Device:C C?
+L Device:C C31
 U 1 1 5E571AEF
 P 5500 1950
-AR Path="/5E564EEA/5E571AEF" Ref="C?"  Part="1"
+AR Path="/5E564EEA/5E571AEF" Ref="C31"  Part="1"
 AR Path="/5E45C906/5E571AEF" Ref="C?"  Part="1"
-F 0 "C?" H 5615 1996 50  0000 L CNN
+F 0 "C31" H 5615 1996 50  0000 L CNN
 F 1 "0.1u" H 5615 1905 50  0000 L CNN
 F 2 "" H 5538 1800 50  0001 C CNN
@@
 $EndComp
 $Comp
-L Device:C C?
+L Device:C C32
 U 1 1 5E571D74
 P 5850 1950
-AR Path="/5E564EEA/5E571D74" Ref="C?"  Part="1"
+AR Path="/5E564EEA/5E571D74" Ref="C32"  Part="1"
 AR Path="/5E45C906/5E571D74" Ref="C?"  Part="1"
-F 0 "C?" H 5965 1996 50  0000 L CNN
+F 0 "C32" H 5965 1996 50  0000 L CNN
 F 1 "4.7u" H 5965 1905 50  0000 L CNN
 F 2 "" H 5888 1800 50  0001 C CNN
@@
 	5850 2200 5500 2200
 $Comp
-L Device:C C?
+L Device:C C33
 U 1 1 5E57AEE1
 P 6300 1950
-AR Path="/5E564EEA/5E57AEE1" Ref="C?"  Part="1"
+AR Path="/5E564EEA/5E57AEE1" Ref="C33"  Part="1"
 AR Path="/5E45C906/5E57AEE1" Ref="C?"  Part="1"
-F 0 "C?" H 6415 1996 50  0000 L CNN
+F 0 "C33" H 6415 1996 50  0000 L CNN
 F 1 "0.1u" H 6415 1905 50  0000 L CNN
 F 2 "" H 6338 1800 50  0001 C CNN
@@
 $EndComp
 $Comp
-L Device:C C?
+L Device:C C34
 U 1 1 5E57B1AF
 P 6650 1950
-AR Path="/5E564EEA/5E57B1AF" Ref="C?"  Part="1"
+AR Path="/5E564EEA/5E57B1AF" Ref="C34"  Part="1"
 AR Path="/5E45C906/5E57B1AF" Ref="C?"  Part="1"
-F 0 "C?" H 6765 1996 50  0000 L CNN
+F 0 "C34" H 6765 1996 50  0000 L CNN
 F 1 "0.1u" H 6765 1905 50  0000 L CNN
 F 2 "" H 6688 1800 50  0001 C CNN
@@
 $EndComp
 $Comp
-L Device:C C?
+L Device:C C35
 U 1 1 5E57B49C
 P 7000 1950
-AR Path="/5E564EEA/5E57B49C" Ref="C?"  Part="1"
+AR Path="/5E564EEA/5E57B49C" Ref="C35"  Part="1"
 AR Path="/5E45C906/5E57B49C" Ref="C?"  Part="1"
-F 0 "C?" H 7115 1996 50  0000 L CNN
+F 0 "C35" H 7115 1996 50  0000 L CNN
 F 1 "4.7u" H 7115 1905 50  0000 L CNN
 F 2 "" H 7038 1800 50  0001 C CNN
@@
 	6300 2200 6300 2100
 $Comp
-L Device:C C?
+L Device:C C36
 U 1 1 5E584EC0
 P 7450 1950
-AR Path="/5E564EEA/5E584EC0" Ref="C?"  Part="1"
+AR Path="/5E564EEA/5E584EC0" Ref="C36"  Part="1"
 AR Path="/5E45C906/5E584EC0" Ref="C?"  Part="1"
-F 0 "C?" H 7565 1996 50  0000 L CNN
+F 0 "C36" H 7565 1996 50  0000 L CNN
 F 1 "10n" H 7565 1905 50  0000 L CNN
 F 2 "" H 7488 1800 50  0001 C CNN
@@
 $EndComp
 $Comp
-L Device:C C?
+L Device:C C37
 U 1 1 5E5855D5
 P 7800 1950
-AR Path="/5E564EEA/5E5855D5" Ref="C?"  Part="1"
+AR Path="/5E564EEA/5E5855D5" Ref="C37"  Part="1"
 AR Path="/5E45C906/5E5855D5" Ref="C?"  Part="1"
-F 0 "C?" H 7915 1996 50  0000 L CNN
+F 0 "C37" H 7915 1996 50  0000 L CNN
 F 1 "1u" H 7915 1905 50  0000 L CNN
 F 2 "" H 7838 1800 50  0001 C CNN
@@
 	7450 1700 7800 1700
 $Comp
-L Device:C C?
+L Device:C C38
 U 1 1 5E5893FA
 P 8200 1950
-AR Path="/5E564EEA/5E5893FA" Ref="C?"  Part="1"
+AR Path="/5E564EEA/5E5893FA" Ref="C38"  Part="1"
 AR Path="/5E45C906/5E5893FA" Ref="C?"  Part="1"
-F 0 "C?" H 8315 1996 50  0000 L CNN
+F 0 "C38" H 8315 1996 50  0000 L CNN
 F 1 "0.1u" H 8315 1905 50  0000 L CNN
 F 2 "" H 8238 1800 50  0001 C CNN
@@
 $EndComp
 $Comp
-L Device:C C?
+L Device:C C39
 U 1 1 5E5897D1
 P 8550 1950
-AR Path="/5E564EEA/5E5897D1" Ref="C?"  Part="1"
+AR Path="/5E564EEA/5E5897D1" Ref="C39"  Part="1"
 AR Path="/5E45C906/5E5897D1" Ref="C?"  Part="1"
-F 0 "C?" H 8665 1996 50  0000 L CNN
+F 0 "C39" H 8665 1996 50  0000 L CNN
 F 1 "4.7u" H 8665 1905 50  0000 L CNN
 F 2 "" H 8588 1800 50  0001 C CNN
@@
 	8400 2200 8200 2200
 $Comp
-L Interface_CAN_LIN:MCP2551-I-SN U?
+L Interface_CAN_LIN:MCP2551-I-SN U5
 U 1 1 5E59148C
 P 7400 4150
-AR Path="/5E564EEA/5E59148C" Ref="U?"  Part="1"
+AR Path="/5E564EEA/5E59148C" Ref="U5"  Part="1"
 AR Path="/5E45C906/5E59148C" Ref="U?"  Part="1"
-F 0 "U?" H 7700 3750 50  0000 C CNN
+F 0 "U5" H 7700 3750 50  0000 C CNN
 F 1 "MCP2551-I-SN" H 7750 3650 50  0000 C CNN
 F 2 "Package_SO:SOIC-8_3.9x4.9mm_P1.27mm" H 7400 3650 50  0001 C CIN
@@
 	7400 4650 7400 4600
 $Comp
-L Device:C C?
+L Device:C C40
 U 1 1 5E596828
 P 7750 3550
-AR Path="/5E564EEA/5E596828" Ref="C?"  Part="1"
+AR Path="/5E564EEA/5E596828" Ref="C40"  Part="1"
 AR Path="/5E45C906/5E596828" Ref="C?"  Part="1"
-F 0 "C?" V 7498 3550 50  0000 C CNN
+F 0 "C40" V 7498 3550 50  0000 C CNN
 F 1 "0.1u" V 7589 3550 50  0000 C CNN
 F 2 "" H 7788 3400 50  0001 C CNN
@@
 	6450 3950 6900 3950
 $Comp
-L Jumper:Jumper_2_Open JP?
+L Jumper:Jumper_2_Open JP1
 U 1 1 5E5AAE77
 P 2700 2600
-AR Path="/5E564EEA/5E5AAE77" Ref="JP?"  Part="1"
+AR Path="/5E564EEA/5E5AAE77" Ref="JP1"  Part="1"
 AR Path="/5E45C906/5E5AAE77" Ref="JP?"  Part="1"
-F 0 "JP?" H 2700 2835 50  0000 C CNN
+F 0 "JP1" H 2700 2835 50  0000 C CNN
 F 1 "Boot Mode" H 2700 2744 50  0000 C CNN
 F 2 "" H 2700 2600 50  0001 C CNN
@@
 $EndComp
 $Comp
-L Device:R_US R?
+L Device:R_US R15
 U 1 1 5E5B42BD
 P 3200 2850
-AR Path="/5E564EEA/5E5B42BD" Ref="R?"  Part="1"
+AR Path="/5E564EEA/5E5B42BD" Ref="R15"  Part="1"
 AR Path="/5E45C906/5E5B42BD" Ref="R?"  Part="1"
-F 0 "R?" H 3268 2896 50  0000 L CNN
+F 0 "R15" H 3268 2896 50  0000 L CNN
 F 1 "510" H 3268 2805 50  0000 L CNN
 F 2 "" V 3240 2840 50  0001 C CNN
@@
 	3200 3100 3200 3000
 $Comp
-L Device:C C?
+L Device:C C28
 U 1 1 5E5BF702
 P 1950 2900
-AR Path="/5E564EEA/5E5BF702" Ref="C?"  Part="1"
+AR Path="/5E564EEA/5E5BF702" Ref="C28"  Part="1"
 AR Path="/5E45C906/5E5BF702" Ref="C?"  Part="1"
-F 0 "C?" H 2065 2946 50  0000 L CNN
+F 0 "C28" H 2065 2946 50  0000 L CNN
 F 1 "18p" H 2065 2855 50  0000 L CNN
 F 2 "" H 1988 2750 50  0001 C CNN
@@
 $EndComp
 $Comp
-L Device:Crystal Y?
+L Device:Crystal Y2
 U 1 1 5E5BFCE2
 P 1650 2550
-AR Path="/5E564EEA/5E5BFCE2" Ref="Y?"  Part="1"
+AR Path="/5E564EEA/5E5BFCE2" Ref="Y2"  Part="1"
 AR Path="/5E45C906/5E5BFCE2" Ref="Y?"  Part="1"
-F 0 "Y?" H 1650 2818 50  0000 C CNN
+F 0 "Y2" H 1650 2818 50  0000 C CNN
 F 1 "16 MHz" H 1650 2727 50  0000 C CNN
 F 2 "" H 1650 2550 50  0001 C CNN
@@
 $EndComp
 $Comp
-L Device:C C?
+L Device:C C27
 U 1 1 5E5C064C
 P 1350 2900
-AR Path="/5E564EEA/5E5C064C" Ref="C?"  Part="1"
+AR Path="/5E564EEA/5E5C064C" Ref="C27"  Part="1"
 AR Path="/5E45C906/5E5C064C" Ref="C?"  Part="1"
-F 0 "C?" H 1465 2946 50  0000 L CNN
+F 0 "C27" H 1465 2946 50  0000 L CNN
 F 1 "18p" H 1465 2855 50  0000 L CNN
 F 2 "" H 1388 2750 50  0001 C CNN
@@
 Connect Jumper\n for Bootloader\n
 $Comp
-L Device:LED D?
+L Device:LED D3
 U 1 1 5E5D4B83
 P 2100 3750
-AR Path="/5E564EEA/5E5D4B83" Ref="D?"  Part="1"
+AR Path="/5E564EEA/5E5D4B83" Ref="D3"  Part="1"
 AR Path="/5E45C906/5E5D4B83" Ref="D?"  Part="1"
-F 0 "D?" V 2139 3633 50  0000 R CNN
+F 0 "D3" V 2139 3633 50  0000 R CNN
 F 1 "LED" V 2048 3633 50  0000 R CNN
 F 2 "" H 2100 3750 50  0001 C CNN
@@
 $EndComp
 $Comp
-L Device:LED D?
+L Device:LED D4
 U 1 1 5E5D53D6
 P 2450 3750
-AR Path="/5E564EEA/5E5D53D6" Ref="D?"  Part="1"
+AR Path="/5E564EEA/5E5D53D6" Ref="D4"  Part="1"
 AR Path="/5E45C906/5E5D53D6" Ref="D?"  Part="1"
-F 0 "D?" V 2489 3633 50  0000 R CNN
+F 0 "D4" V 2489 3633 50  0000 R CNN
 F 1 "LED" V 2398 3633 50  0000 R CNN
 F 2 "" H 2450 3750 50  0001 C CNN
@@
 	3500 3300 3750 3300
 $Comp
-L Device:R_US R?
+L Device:R_US R13
 U 1 1 5E5DDB72
 P 2100 4150
-AR Path="/5E564EEA/5E5DDB72" Ref="R?"  Part="1"
+AR Path="/5E564EEA/5E5DDB72" Ref="R13"  Part="1"
 AR Path="/5E45C906/5E5DDB72" Ref="R?"  Part="1"
-F 0 "R?" H 2168 4196 50  0000 L CNN
+F 0 "R13" H 2168 4196 50  0000 L CNN
 F 1 "120" H 2168 4105 50  0000 L CNN
 F 2 "" V 2140 4140 50  0001 C CNN
@@
 $EndComp
 $Comp
-L Device:R_US R?
+L Device:R_US R14
 U 1 1 5E5DE222
 P 2450 4150
-AR Path="/5E564EEA/5E5DE222" Ref="R?"  Part="1"
+AR Path="/5E564EEA/5E5DE222" Ref="R14"  Part="1"
 AR Path="/5E45C906/5E5DE222" Ref="R?"  Part="1"
-F 0 "R?" H 2518 4196 50  0000 L CNN
+F 0 "R14" H 2518 4196 50  0000 L CNN
 F 1 "120" H 2518 4105 50  0000 L CNN
 F 2 "" V 2490 4140 50  0001 C CNN
@@
 	2250 4450 2100 4450
 $Comp
-L Device:R_US R?
+L Device:R_US R16
 U 1 1 5E5FF6DC
 P 8750 4250
-AR Path="/5E564EEA/5E5FF6DC" Ref="R?"  Part="1"
+AR Path="/5E564EEA/5E5FF6DC" Ref="R16"  Part="1"
 AR Path="/5E45C906/5E5FF6DC" Ref="R?"  Part="1"
-F 0 "R?" H 8818 4296 50  0000 L CNN
+F 0 "R16" H 8818 4296 50  0000 L CNN
 F 1 "120" H 8818 4205 50  0000 L CNN
 F 2 "" V 8790 4240 50  0001 C CNN
