File: Hardware/USB_HEADERS.sch (KiCad schematic (older format))
At the start: 1 part, among them J5 USB Headers Board Top

Commit message: Added footprints to schematic symbols
Parts:
- J5: footprint (none) -> Connector_PinHeader_2.54mm:PinHeader_2x04_P2.54mm_Vertical_SMD; symbol Connector_Generic:Conn_02x04_Counter_Clockwise -> Connector_Generic:Conn_02x04_Odd_Even
Connections:
- net BOARD_5V: now also J5.2 (Pin_2), J5.8 (Pin_8); no longer J5.5 (Pin_5)
- net USB_DM: now also J5.4 (Pin_4); no longer J5.7 (Pin_7)
- removed net BOARD_GND: J5.1 (Pin_1), J5.2 (Pin_2), J5.3 (Pin_3), J5.4 (Pin_4), J5.8 (Pin_8)
- new net: J5.1 (Pin_1), J5.3 (Pin_3), J5.5 (Pin_5), J5.7 (Pin_7)
Other:
- moved on the sheet: J5
Changed lines of the file:
@@
 $EndDescr
 $Comp
-L Connector_Generic:Conn_02x04_Counter_Clockwise J5
+L Connector_Generic:Conn_02x04_Odd_Even J5
 U 1 1 5E532F04
-P 4150 1950
-F 0 "J5" H 4200 2267 50  0000 C CNN
-F 1 "USB Headers Board Top" H 4200 2176 50  0000 C CNN
-F 2 "" H 4150 1950 50  0001 C CNN
-F 3 "~" H 4150 1950 50  0001 C CNN
-	1    4150 1950
+P 4150 2050
+F 0 "J5" H 4200 1550 50  0000 C CNN
+F 1 "USB Headers Board Top" H 4200 1400 50  0000 C CNN
+F 2 "Connector_PinHeader_2.54mm:PinHeader_2x04_P2.54mm_Vertical_SMD" H 4150 2050 50  0001 C CNN
+F 3 "~" H 4150 2050 50  0001 C CNN
+	1    4150 2050
 	1    0    0    -1
 $EndComp
-Text Notes 4500 1850 0    50   ~ 0
-GND
-Text Notes 3750 1850 0    50   ~ 0
+Text Notes 4500 1950 0    50   ~ 0
 GND
 Text Notes 3750 1950 0    50   ~ 0
@@
 Text Notes 3750 2150 0    50   ~ 0
 GND
-Text Notes 4500 1950 0    50   ~ 0
+Text Notes 3750 2250 0    50   ~ 0
+GND
+Text Notes 4500 2050 0    50   ~ 0
 D-
-Text Notes 4500 2050 0    50   ~ 0
+Text Notes 4500 2150 0    50   ~ 0
 D+
-Text Notes 4500 2150 0    50   ~ 0
+Text Notes 4500 2250 0    50   ~ 0
 5V
-Text HLabel 4800 1950 2    50   Input ~ 0
+Text HLabel 4800 2050 2    50   Input ~ 0
 USB_DM
-Text HLabel 4800 2050 2    50   Input ~ 0
+Text HLabel 4800 2150 2    50   Input ~ 0
 USB_DP
 Wire Wire Line
-	4800 1950 4450 1950
+	4800 2050 4450 2050
 Wire Wire Line
-	4800 2050 4450 2050
-Text HLabel 4800 2150 2    50   Input ~ 0
+	4800 2150 4450 2150
+Text HLabel 4800 2250 2    50   Input ~ 0
 BOARD_5V
-Text HLabel 4800 1850 2    50   Input ~ 0
+Text HLabel 4800 1950 2    50   Input ~ 0
 BOARD_GND
 Wire Wire Line
-	4800 1850 4700 1850
-Wire Wire Line
-	4800 2150 4450 2150
-Wire Wire Line
-	4700 1850 4700 1550
-Wire Wire Line
-	4700 1550 3700 1550
-Wire Wire Line
-	3700 1550 3700 1850
-Wire Wire Line
-	3700 1850 3950 1850
-Connection ~ 4700 1850
-Wire Wire Line
-	4700 1850 4450 1850
-Wire Wire Line
-	3700 1850 3700 1950
+	4800 2250 4700 2250
 Wire Wire Line
 	3700 1950 3950 1950
-Connection ~ 3700 1850
+Wire Wire Line
+	4700 1950 4450 1950
+Wire Wire Line
+	3700 2050 3950 2050
 Wire Wire Line
 	3700 1950 3700 2050
 Wire Wire Line
-	3700 2050 3950 2050
-Connection ~ 3700 1950
+	3700 2150 3950 2150
 Wire Wire Line
 	3700 2050 3700 2150
 Wire Wire Line
-	3700 2150 3950 2150
+	3700 2250 3950 2250
 Connection ~ 3700 2050
+Wire Wire Line
+	3700 2250 3700 2150
+Connection ~ 3700 2150
+Connection ~ 4700 2250
+Wire Wire Line
+	4700 2250 4450 2250
+Connection ~ 4700 1950
+Wire Wire Line
+	4700 1950 4700 2250
+Wire Wire Line
+	4700 1950 4800 1950
 $EndSCHEMATC
