File: Hardware/lattepanda.sch (KiCad schematic (older format))
At the start: 17 parts, among them J10 Lattepanda Lower Left Header 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, J6 Lattepanda Upper Left Header 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, J7 Lattepanda Upper Right Header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, J8 Lattepanda Middle Left Header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, J9 Lattepanda Lower Right Header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, U7 TLC59108xPW

Commit message: Added footprints to schematic symbols
Parts:
- added J11: 12V DC IN Headers, Connector_PinHeader_2.54mm:PinHeader_2x02_P2.54mm_Vertical, symbol Connector_Generic:Conn_02x02_Odd_Even
- D10, D11, D12, D13, D14, D7, D8, D9: footprint (none) -> LED_SMD:LED_0805_2012Metric_Castellated
- J10: footprint Connector_PinHeader_2.00mm:PinHeader_2x06_P2.00mm_Vertical_SMD -> Connector_PinHeader_2.54mm:PinHeader_2x06_P2.54mm_Vertical_SMD; symbol Connector_Generic:Conn_02x06_Odd_Even -> Connector_Generic:Conn_02x04_Odd_Even
- J6: footprint Connector_PinHeader_2.00mm:PinHeader_2x12_P2.00mm_Vertical_SMD -> Connector_PinHeader_2.54mm:PinHeader_2x12_P2.54mm_Vertical
- J7: footprint Connector_PinHeader_2.00mm:PinHeader_2x09_P2.00mm_Vertical_SMD -> Connector_PinHeader_2.54mm:PinHeader_2x09_P2.54mm_Vertical
- J8: footprint Connector_PinHeader_2.00mm:PinHeader_2x05_P2.00mm_Vertical_SMD -> Connector_PinHeader_2.54mm:PinHeader_2x05_P2.54mm_Vertical
- J9: footprint Connector_PinHeader_2.00mm:PinHeader_2x15_P2.00mm_Vertical_SMD -> Connector_PinHeader_2.54mm:PinHeader_2x15_P2.54mm_Vertical
- R21, R22, R23: footprint (none) -> Resistor_SMD:R_1206_3216Metric
- renumbered U7 to U8
Changed lines of the file:
@@
 F 0 "J9" H 4150 4467 50  0000 C CNN
 F 1 "Lattepanda Lower Right Header (Arduino Pins)" H 4150 4376 50  0000 C CNN
-F 2 "Connector_PinHeader_2.00mm:PinHeader_2x15_P2.00mm_Vertical_SMD" H 4100 3550 50  0001 C CNN
+F 2 "Connector_PinHeader_2.54mm:PinHeader_2x15_P2.54mm_Vertical" H 4100 3550 50  0001 C CNN
 F 3 "~" H 4100 3550 50  0001 C CNN
 	1    4100 3550
@@
 F 0 "J8" H 2350 3517 50  0000 C CNN
 F 1 "Lattepanda Middle Left Header (RS-232)" H 2350 3426 50  0000 C CNN
-F 2 "Connector_PinHeader_2.00mm:PinHeader_2x05_P2.00mm_Vertical_SMD" H 2300 3100 50  0001 C CNN
+F 2 "Connector_PinHeader_2.54mm:PinHeader_2x05_P2.54mm_Vertical" H 2300 3100 50  0001 C CNN
 F 3 "~" H 2300 3100 50  0001 C CNN
 	1    2300 3100
@@
 Text Notes 2650 3300 0    50   ~ 0
 DCD
-$Comp
-L Connector_Generic:Conn_02x06_Odd_Even J10
-U 1 1 5E4824AD
-P 2300 3900
-F 0 "J10" H 2350 4317 50  0000 C CNN
-F 1 "Lattepanda Lower Left Header (USB)" H 2350 4226 50  0000 C CNN
-F 2 "Connector_PinHeader_2.00mm:PinHeader_2x06_P2.00mm_Vertical_SMD" H 2300 3900 50  0001 C CNN
-F 3 "~" H 2300 3900 50  0001 C CNN
-	1    2300 3900
-	1    0    0    -1
-$EndComp
 Text Notes 1900 3700 0    50   ~ 0
 GND
@@
 Text Notes 1900 4000 0    50   ~ 0
 GND
-Text Notes 1900 4100 0    50   ~ 0
-GND
-Text Notes 1900 4200 0    50   ~ 0
+Text Notes 1900 4350 0    50   ~ 0
+GND
+Text Notes 1900 4450 0    50   ~ 0
 GND
 Text Notes 2650 3700 0    50   ~ 0
@@
 Text Notes 2650 4000 0    50   ~ 0
 5V
-Text Notes 2650 4100 0    50   ~ 0
+Text Notes 2650 4350 0    50   ~ 0
 DC_IN
-Text Notes 2650 4200 0    50   ~ 0
+Text Notes 2650 4450 0    50   ~ 0
 DC_IN
 $Comp
@@
 F 0 "J7" H 4150 2417 50  0000 C CNN
 F 1 "Lattepanda Upper Right Header (BIOS SPI)" H 4150 2326 50  0000 C CNN
-F 2 "Connector_PinHeader_2.00mm:PinHeader_2x09_P2.00mm_Vertical_SMD" H 4100 1800 50  0001 C CNN
+F 2 "Connector_PinHeader_2.54mm:PinHeader_2x09_P2.54mm_Vertical" H 4100 1800 50  0001 C CNN
 F 3 "~" H 4100 1800 50  0001 C CNN
 	1    4100 1800
@@
 F 0 "J6" H 2350 2617 50  0000 C CNN
 F 1 "Lattepanda Upper Left Header (I2C and I2S)" H 2350 2526 50  0000 C CNN
-F 2 "Connector_PinHeader_2.00mm:PinHeader_2x12_P2.00mm_Vertical_SMD" H 2300 1900 50  0001 C CNN
+F 2 "Connector_PinHeader_2.54mm:PinHeader_2x12_P2.54mm_Vertical" H 2300 1900 50  0001 C CNN
 F 3 "~" H 2300 1900 50  0001 C CNN
 	1    2300 1900
@@
 F 0 "R22" H 5368 2096 50  0000 L CNN
 F 1 "4.7k" H 5368 2005 50  0000 L CNN
-F 2 "" V 5340 2040 50  0001 C CNN
+F 2 "Resistor_SMD:R_1206_3216Metric" V 5340 2040 50  0001 C CNN
 F 3 "~" H 5300 2050 50  0001 C CNN
 	1    5300 2050
@@
 F 0 "R21" H 5018 2096 50  0000 L CNN
 F 1 "4.7k" H 5018 2005 50  0000 L CNN
-F 2 "" V 4990 2040 50  0001 C CNN
+F 2 "Resistor_SMD:R_1206_3216Metric" V 4990 2040 50  0001 C CNN
 F 3 "~" H 4950 2050 50  0001 C CNN
 	1    4950 2050
@@
 	3350 2300 4950 2300
 $Comp
-L Driver_LED:TLC59108xPW U7
+L Driver_LED:TLC59108xPW U8
 U 1 1 5E4AC79A
 P 6300 2600
-F 0 "U7" H 5900 3300 50  0000 C CNN
+F 0 "U8" H 5900 3300 50  0000 C CNN
 F 1 "TLC59108xPW" H 5900 3200 50  0000 C CNN
 F 2 "Package_SO:TSSOP-20_4.4x6.5mm_P0.65mm" H 6300 2600 50  0001 C CNN
@@
 F 0 "D7" V 7539 1933 50  0000 R CNN
 F 1 "LED" V 7448 1933 50  0000 R CNN
-F 2 "" H 7500 2050 50  0001 C CNN
+F 2 "LED_SMD:LED_0805_2012Metric_Castellated" H 7500 2050 50  0001 C CNN
 F 3 "~" H 7500 2050 50  0001 C CNN
 	1    7500 2050
@@
 F 0 "D8" V 7889 1933 50  0000 R CNN
 F 1 "LED" V 7798 1933 50  0000 R CNN
-F 2 "" H 7850 2050 50  0001 C CNN
+F 2 "LED_SMD:LED_0805_2012Metric_Castellated" H 7850 2050 50  0001 C CNN
 F 3 "~" H 7850 2050 50  0001 C CNN
 	1    7850 2050
@@
 F 0 "D9" V 8189 1933 50  0000 R CNN
 F 1 "LED" V 8098 1933 50  0000 R CNN
-F 2 "" H 8150 2050 50  0001 C CNN
+F 2 "LED_SMD:LED_0805_2012Metric_Castellated" H 8150 2050 50  0001 C CNN
 F 3 "~" H 8150 2050 50  0001 C CNN
 	1    8150 2050
@@
 F 0 "D10" V 8489 1932 50  0000 R CNN
 F 1 "LED" V 8398 1932 50  0000 R CNN
-F 2 "" H 8450 2050 50  0001 C CNN
+F 2 "LED_SMD:LED_0805_2012Metric_Castellated" H 8450 2050 50  0001 C CNN
 F 3 "~" H 8450 2050 50  0001 C CNN
 	1    8450 2050
@@
 F 0 "D11" V 8789 1932 50  0000 R CNN
 F 1 "LED" V 8698 1932 50  0000 R CNN
-F 2 "" H 8750 2050 50  0001 C CNN
+F 2 "LED_SMD:LED_0805_2012Metric_Castellated" H 8750 2050 50  0001 C CNN
 F 3 "~" H 8750 2050 50  0001 C CNN
 	1    8750 2050
@@
 F 0 "D12" V 9089 1932 50  0000 R CNN
 F 1 "LED" V 8998 1932 50  0000 R CNN
-F 2 "" H 9050 2050 50  0001 C CNN
+F 2 "LED_SMD:LED_0805_2012Metric_Castellated" H 9050 2050 50  0001 C CNN
 F 3 "~" H 9050 2050 50  0001 C CNN
 	1    9050 2050
@@
 F 0 "D13" V 9389 1932 50  0000 R CNN
 F 1 "LED" V 9298 1932 50  0000 R CNN
-F 2 "" H 9350 2050 50  0001 C CNN
+F 2 "LED_SMD:LED_0805_2012Metric_Castellated" H 9350 2050 50  0001 C CNN
 F 3 "~" H 9350 2050 50  0001 C CNN
 	1    9350 2050
@@
 F 0 "D14" V 9689 1932 50  0000 R CNN
 F 1 "LED" V 9598 1932 50  0000 R CNN
-F 2 "" H 9650 2050 50  0001 C CNN
+F 2 "LED_SMD:LED_0805_2012Metric_Castellated" H 9650 2050 50  0001 C CNN
 F 3 "~" H 9650 2050 50  0001 C CNN
 	1    9650 2050
@@
 F 0 "R23" H 5368 3196 50  0000 L CNN
 F 1 "4.7k" H 5368 3105 50  0000 L CNN
-F 2 "" V 5340 3140 50  0001 C CNN
+F 2 "Resistor_SMD:R_1206_3216Metric" V 5340 3140 50  0001 C CNN
 F 3 "~" H 5300 3150 50  0001 C CNN
 	1    5300 3150
@@
 	5600 2800 5600 3450
 $Comp
-L power:GNDREF #PWR?
+L power:GNDREF #PWR0181
 U 1 1 5E4FCB1D
 P 5600 3600
-F 0 "#PWR?" H 5600 3350 50  0001 C CNN
+F 0 "#PWR0181" H 5600 3350 50  0001 C CNN
 F 1 "GNDREF" H 5605 3427 50  0000 C CNN
 F 2 "" H 5600 3600 50  0001 C CNN
@@
 Wire Wire Line
 	6800 2600 8750 2600
+$Comp
+L Connector_Generic:Conn_02x02_Odd_Even J11
+U 1 1 5E51EE90
+P 2300 4350
+F 0 "J11" H 2350 4567 50  0000 C CNN
+F 1 "12V DC IN Headers" H 2350 4476 50  0000 C CNN
+F 2 "Connector_PinHeader_2.54mm:PinHeader_2x02_P2.54mm_Vertical" H 2300 4350 50  0001 C CNN
+F 3 "~" H 2300 4350 50  0001 C CNN
+	1    2300 4350
+	1    0    0    -1
+$EndComp
+$Comp
+L Connector_Generic:Conn_02x04_Odd_Even J10
+U 1 1 5E4824AD
+P 2300 3800
+F 0 "J10" H 2350 4150 50  0000 C CNN
+F 1 "Lattepanda Lower Left Header (USB)" H 2350 4050 50  0000 C CNN
+F 2 "Connector_PinHeader_2.54mm:PinHeader_2x06_P2.54mm_Vertical_SMD" H 2300 3800 50  0001 C CNN
+F 3 "~" H 2300 3800 50  0001 C CNN
+	1    2300 3800
+	1    0    0    -1
+$EndComp
 $EndSCHEMATC
