File: hardware/avenashield/LTE_Modem.sch (KiCad schematic (older format))
At the start: 19 parts, among them J1 Bus_PCI_Express_Mini, J2 SIM_Card

Commit message: Changed footprints for CAN connectors and replaced 3D models for headers
Parts:
- C13, C14, C16, C17: footprint Capacitor_SMD:C_1206_3216Metric_Pad1.42x1.75mm_HandSolder -> Capacitor_SMD:C_0805_2012Metric_Pad1.15x1.40mm_HandSolder
- C15, C18, C19, C20, C21, C22: footprint Capacitor_SMD:C_0603_1608Metric_Pad1.05x0.95mm_HandSolder -> Capacitor_SMD:C_0805_2012Metric_Pad1.15x1.40mm_HandSolder
- R10, R11, R12, R8, R9: footprint Resistor_SMD:R_1206_3216Metric -> Resistor_SMD:R_0805_2012Metric_Pad1.15x1.40mm_HandSolder
Changed lines of the file:
@@
 F 0 "C19" H 7815 5246 50  0000 L CNN
 F 1 "100n" H 7815 5155 50  0000 L CNN
-F 2 "Capacitor_SMD:C_0603_1608Metric_Pad1.05x0.95mm_HandSolder" H 7738 5050 50  0001 C CNN
+F 2 "Capacitor_SMD:C_0805_2012Metric_Pad1.15x1.40mm_HandSolder" H 7738 5050 50  0001 C CNN
 F 3 "~" H 7700 5200 50  0001 C CNN
 	1    7700 5200
@@
 F 0 "C20" H 8315 5246 50  0000 L CNN
 F 1 "33p" H 8315 5155 50  0000 L CNN
-F 2 "Capacitor_SMD:C_0603_1608Metric_Pad1.05x0.95mm_HandSolder" H 8238 5050 50  0001 C CNN
+F 2 "Capacitor_SMD:C_0805_2012Metric_Pad1.15x1.40mm_HandSolder" H 8238 5050 50  0001 C CNN
 F 3 "~" H 8200 5200 50  0001 C CNN
 	1    8200 5200
@@
 F 0 "C21" H 8815 5246 50  0000 L CNN
 F 1 "33p" H 8815 5155 50  0000 L CNN
-F 2 "Capacitor_SMD:C_0603_1608Metric_Pad1.05x0.95mm_HandSolder" H 8738 5050 50  0001 C CNN
+F 2 "Capacitor_SMD:C_0805_2012Metric_Pad1.15x1.40mm_HandSolder" H 8738 5050 50  0001 C CNN
 F 3 "~" H 8700 5200 50  0001 C CNN
 	1    8700 5200
@@
 F 0 "C22" H 9215 5246 50  0000 L CNN
 F 1 "33p" H 9215 5155 50  0000 L CNN
-F 2 "Capacitor_SMD:C_0603_1608Metric_Pad1.05x0.95mm_HandSolder" H 9138 5050 50  0001 C CNN
+F 2 "Capacitor_SMD:C_0805_2012Metric_Pad1.15x1.40mm_HandSolder" H 9138 5050 50  0001 C CNN
 F 3 "~" H 9100 5200 50  0001 C CNN
 	1    9100 5200
@@
 F 0 "R10" V 6450 4100 50  0000 C CNN
 F 1 "47" V 6450 4500 50  0000 C CNN
-F 2 "Resistor_SMD:R_1206_3216Metric" V 6540 4290 50  0001 C CNN
+F 2 "Resistor_SMD:R_0805_2012Metric_Pad1.15x1.40mm_HandSolder" V 6540 4290 50  0001 C CNN
 F 3 "~" H 6500 4300 50  0001 C CNN
 	1    6500 4300
@@
 F 0 "R11" V 6450 4200 50  0000 C CNN
 F 1 "47" V 6450 4600 50  0000 C CNN
-F 2 "Resistor_SMD:R_1206_3216Metric" V 6540 4390 50  0001 C CNN
+F 2 "Resistor_SMD:R_0805_2012Metric_Pad1.15x1.40mm_HandSolder" V 6540 4390 50  0001 C CNN
 F 3 "~" H 6500 4400 50  0001 C CNN
 	1    6500 4400
@@
 F 0 "R12" V 6450 4300 50  0000 C CNN
 F 1 "47" V 6450 4700 50  0000 C CNN
-F 2 "Resistor_SMD:R_1206_3216Metric" V 6540 4490 50  0001 C CNN
+F 2 "Resistor_SMD:R_0805_2012Metric_Pad1.15x1.40mm_HandSolder" V 6540 4490 50  0001 C CNN
 F 3 "~" H 6500 4500 50  0001 C CNN
 	1    6500 4500
@@
 F 0 "R9" V 6245 3100 50  0000 C CNN
 F 1 "330" V 6336 3100 50  0000 C CNN
-F 2 "Resistor_SMD:R_1206_3216Metric" V 6490 3090 50  0001 C CNN
+F 2 "Resistor_SMD:R_0805_2012Metric_Pad1.15x1.40mm_HandSolder" V 6490 3090 50  0001 C CNN
 F 3 "~" H 6450 3100 50  0001 C CNN
 	1    6450 3100
@@
 F 0 "C13" H 1965 2546 50  0000 L CNN
 F 1 "100u" H 1965 2455 50  0000 L CNN
-F 2 "Capacitor_SMD:C_1206_3216Metric_Pad1.42x1.75mm_HandSolder" H 1888 2350 50  0001 C CNN
+F 2 "Capacitor_SMD:C_0805_2012Metric_Pad1.15x1.40mm_HandSolder" H 1888 2350 50  0001 C CNN
 F 3 "~" H 1850 2500 50  0001 C CNN
 	1    1850 2500
@@
 F 0 "C14" H 2415 2546 50  0000 L CNN
 F 1 "100u" H 2415 2455 50  0000 L CNN
-F 2 "Capacitor_SMD:C_1206_3216Metric_Pad1.42x1.75mm_HandSolder" H 2338 2350 50  0001 C CNN
+F 2 "Capacitor_SMD:C_0805_2012Metric_Pad1.15x1.40mm_HandSolder" H 2338 2350 50  0001 C CNN
 F 3 "~" H 2300 2500 50  0001 C CNN
 	1    2300 2500
@@
 F 0 "C15" H 2815 2546 50  0000 L CNN
 F 1 "100n" H 2815 2455 50  0000 L CNN
-F 2 "Capacitor_SMD:C_0603_1608Metric_Pad1.05x0.95mm_HandSolder" H 2738 2350 50  0001 C CNN
+F 2 "Capacitor_SMD:C_0805_2012Metric_Pad1.15x1.40mm_HandSolder" H 2738 2350 50  0001 C CNN
 F 3 "~" H 2700 2500 50  0001 C CNN
 	1    2700 2500
@@
 F 0 "C16" H 3265 2546 50  0000 L CNN
 F 1 "100u" H 3265 2455 50  0000 L CNN
-F 2 "Capacitor_SMD:C_1206_3216Metric_Pad1.42x1.75mm_HandSolder" H 3188 2350 50  0001 C CNN
+F 2 "Capacitor_SMD:C_0805_2012Metric_Pad1.15x1.40mm_HandSolder" H 3188 2350 50  0001 C CNN
 F 3 "~" H 3150 2500 50  0001 C CNN
 	1    3150 2500
@@
 F 0 "C17" H 3715 2546 50  0000 L CNN
 F 1 "100u" H 3715 2455 50  0000 L CNN
-F 2 "Capacitor_SMD:C_1206_3216Metric_Pad1.42x1.75mm_HandSolder" H 3638 2350 50  0001 C CNN
+F 2 "Capacitor_SMD:C_0805_2012Metric_Pad1.15x1.40mm_HandSolder" H 3638 2350 50  0001 C CNN
 F 3 "~" H 3600 2500 50  0001 C CNN
 	1    3600 2500
@@
 F 0 "C18" H 4165 2546 50  0000 L CNN
 F 1 "100n" H 4165 2455 50  0000 L CNN
-F 2 "Capacitor_SMD:C_0603_1608Metric_Pad1.05x0.95mm_HandSolder" H 4088 2350 50  0001 C CNN
+F 2 "Capacitor_SMD:C_0805_2012Metric_Pad1.15x1.40mm_HandSolder" H 4088 2350 50  0001 C CNN
 F 3 "~" H 4050 2500 50  0001 C CNN
 	1    4050 2500
@@
 F 0 "R8" H 1718 3596 50  0000 L CNN
 F 1 "330" H 1718 3505 50  0000 L CNN
-F 2 "Resistor_SMD:R_1206_3216Metric" V 1690 3540 50  0001 C CNN
+F 2 "Resistor_SMD:R_0805_2012Metric_Pad1.15x1.40mm_HandSolder" V 1690 3540 50  0001 C CNN
 F 3 "~" H 1650 3550 50  0001 C CNN
 	1    1650 3550
