File: hardware/avenashield/USB_HUB.sch (KiCad schematic (older format))
At the start: 23 parts, among them U1 USB2514B_Bi, U2 MIC2026-1BM, U3 MIC2026-1BM, Y1 24 MHz

Commit message: Changed footprints for CAN connectors and replaced 3D models for headers
Parts:
- C1, C10, C11, C12, C2, C3, C4, C5, C6, C7, C8, C9: footprint Capacitor_SMD:C_0603_1608Metric -> Capacitor_SMD:C_0805_2012Metric_Pad1.15x1.40mm_HandSolder
Changed lines of the file:
@@
 F 0 "C1" V 1748 2950 50  0000 C CNN
 F 1 "18pF" V 1839 2950 50  0000 C CNN
-F 2 "Capacitor_SMD:C_0603_1608Metric" H 2038 2800 50  0001 C CNN
+F 2 "Capacitor_SMD:C_0805_2012Metric_Pad1.15x1.40mm_HandSolder" H 2038 2800 50  0001 C CNN
 F 3 "~" H 2000 2950 50  0001 C CNN
 	1    2000 2950
@@
 F 0 "C2" V 1748 3400 50  0000 C CNN
 F 1 "18pF" V 1839 3400 50  0000 C CNN
-F 2 "Capacitor_SMD:C_0603_1608Metric" H 2038 3250 50  0001 C CNN
+F 2 "Capacitor_SMD:C_0805_2012Metric_Pad1.15x1.40mm_HandSolder" H 2038 3250 50  0001 C CNN
 F 3 "~" H 2000 3400 50  0001 C CNN
 	1    2000 3400
@@
 F 0 "C3" H 2315 3946 50  0000 L CNN
 F 1 "0.1uF" H 2315 3855 50  0000 L CNN
-F 2 "Capacitor_SMD:C_0603_1608Metric" H 2238 3750 50  0001 C CNN
+F 2 "Capacitor_SMD:C_0805_2012Metric_Pad1.15x1.40mm_HandSolder" H 2238 3750 50  0001 C CNN
 F 3 "~" H 2200 3900 50  0001 C CNN
 	1    2200 3900
@@
 F 0 "C4" H 2815 3946 50  0000 L CNN
 F 1 "0.1uF" H 2815 3855 50  0000 L CNN
-F 2 "Capacitor_SMD:C_0603_1608Metric" H 2738 3750 50  0001 C CNN
+F 2 "Capacitor_SMD:C_0805_2012Metric_Pad1.15x1.40mm_HandSolder" H 2738 3750 50  0001 C CNN
 F 3 "~" H 2700 3900 50  0001 C CNN
 	1    2700 3900
@@
 F 0 "C5" H 915 1396 50  0000 L CNN
 F 1 "0.1uF" H 915 1305 50  0000 L CNN
-F 2 "Capacitor_SMD:C_0603_1608Metric" H 838 1200 50  0001 C CNN
+F 2 "Capacitor_SMD:C_0805_2012Metric_Pad1.15x1.40mm_HandSolder" H 838 1200 50  0001 C CNN
 F 3 "~" H 800 1350 50  0001 C CNN
 	1    800  1350
@@
 F 0 "C6" H 1365 1396 50  0000 L CNN
 F 1 "0.1uF" H 1365 1305 50  0000 L CNN
-F 2 "Capacitor_SMD:C_0603_1608Metric" H 1288 1200 50  0001 C CNN
+F 2 "Capacitor_SMD:C_0805_2012Metric_Pad1.15x1.40mm_HandSolder" H 1288 1200 50  0001 C CNN
 F 3 "~" H 1250 1350 50  0001 C CNN
 	1    1250 1350
@@
 F 0 "C7" H 1815 1396 50  0000 L CNN
 F 1 "0.1uF" H 1815 1305 50  0000 L CNN
-F 2 "Capacitor_SMD:C_0603_1608Metric" H 1738 1200 50  0001 C CNN
+F 2 "Capacitor_SMD:C_0805_2012Metric_Pad1.15x1.40mm_HandSolder" H 1738 1200 50  0001 C CNN
 F 3 "~" H 1700 1350 50  0001 C CNN
 	1    1700 1350
@@
 F 0 "C8" H 2265 1396 50  0000 L CNN
 F 1 "0.1uF" H 2265 1305 50  0000 L CNN
-F 2 "Capacitor_SMD:C_0603_1608Metric" H 2188 1200 50  0001 C CNN
+F 2 "Capacitor_SMD:C_0805_2012Metric_Pad1.15x1.40mm_HandSolder" H 2188 1200 50  0001 C CNN
 F 3 "~" H 2150 1350 50  0001 C CNN
 	1    2150 1350
@@
 F 0 "C9" H 1365 3046 50  0000 L CNN
 F 1 "0.1uF" H 1365 2955 50  0000 L CNN
-F 2 "Capacitor_SMD:C_0603_1608Metric" H 1288 2850 50  0001 C CNN
+F 2 "Capacitor_SMD:C_0805_2012Metric_Pad1.15x1.40mm_HandSolder" H 1288 2850 50  0001 C CNN
 F 3 "~" H 1250 3000 50  0001 C CNN
 	1    1250 3000
@@
 F 0 "C10" H 2715 1396 50  0000 L CNN
 F 1 "0.1uF" H 2715 1305 50  0000 L CNN
-F 2 "Capacitor_SMD:C_0603_1608Metric" H 2638 1200 50  0001 C CNN
+F 2 "Capacitor_SMD:C_0805_2012Metric_Pad1.15x1.40mm_HandSolder" H 2638 1200 50  0001 C CNN
 F 3 "~" H 2600 1350 50  0001 C CNN
 	1    2600 1350
@@
 F 0 "C11" H 3165 1396 50  0000 L CNN
 F 1 "0.1uF" H 3165 1305 50  0000 L CNN
-F 2 "Capacitor_SMD:C_0603_1608Metric" H 3088 1200 50  0001 C CNN
+F 2 "Capacitor_SMD:C_0805_2012Metric_Pad1.15x1.40mm_HandSolder" H 3088 1200 50  0001 C CNN
 F 3 "~" H 3050 1350 50  0001 C CNN
 	1    3050 1350
@@
 F 0 "C12" H 3615 1396 50  0000 L CNN
 F 1 "4.7uF" H 3615 1305 50  0000 L CNN
-F 2 "Capacitor_SMD:C_0603_1608Metric" H 3538 1200 50  0001 C CNN
+F 2 "Capacitor_SMD:C_0805_2012Metric_Pad1.15x1.40mm_HandSolder" H 3538 1200 50  0001 C CNN
 F 3 "~" H 3500 1350 50  0001 C CNN
 	1    3500 1350
