File: hardware/avenashield/avenashield.kicad_pcb (KiCad board)
At the start: 4 copper layers, 115 x 78 mm, 124 parts, among them J1 MiniPCIe LTE Modem, J10 Lattepanda Lower Left Header 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, J11 12V DC IN Headers, J2 SIM_Card, J3 CAN_TRA_HEADER, J4 CAN_IMP_HEADER, J5 USB Headers Board Top, J6 Lattepanda Upper Left Header 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, J7 Lattepanda Upper Right Header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, J8 Lattepanda Middle Left Header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

Commit message: Added MiniPCIe latch clip and replaced onboard LEDs with connector
Parts:
- removed D10, D11, D12, D13, D14, D7, D8, D9: LED, LED_SMD:LED_0805_2012Metric_Castellated
- removed SW1: CAN 1 ON/OFF, Button_Switch_SMD:SW_MEC_5GSH9
- removed SW2: CAN 2 ON/OFF, Button_Switch_SMD:SW_MEC_5GSH9
- added G***: PURDUE_LOGO, Images:PURDUE_LOGO, F.Cu at (67.3, 90.8)
- added G***: OATS_LOGO, Images:OATS_LOGO, F.Cu at (68.7, 86.8)
- added H1: MOUNT_PAD1, MountingHole:MountingHole_3.2mm_M3_Pad_Via, F.Cu at (55.7, 82.7)
- added H2: MOUNT_PAD2, MountingHole:MountingHole_3.2mm_M3_Pad_Via, F.Cu at (55.7, 152.6)
- added H3: MOUNT_PAD3, MountingHole:MountingHole_3.2mm_M3_Pad_Via, F.Cu at (162.7, 82.7)
- added H4: MOUNT_PAD4, MountingHole:MountingHole_3.2mm_M3_Pad_Via, F.Cu at (162.7, 152.6)
- added J12: EXT PWR IN, Connector_PinHeader_2.54mm:PinHeader_2x02_P2.54mm_Vertical, F.Cu at (147.0, 150.3)
- added J13: LED_OUT, Connector_PinHeader_2.54mm:PinHeader_2x05_P2.54mm_Horizontal, F.Cu at (66.1, 106.8)
- added JP5: 3.3V SRC SEL, Connector_PinHeader_2.54mm:PinHeader_1x03_P2.54mm_Vertical_SMD_Pin1Left, F.Cu at (158.9, 143.8)
- added JP6: 5V SRC SEL, Connector_PinHeader_2.54mm:PinHeader_1x03_P2.54mm_Vertical_SMD_Pin1Left, F.Cu at (149.0, 143.7)
- added R26: 200k, Resistor_SMD:R_0805_2012Metric_Pad1.15x1.40mm_HandSolder, B.Cu at (125.6, 93.9)
- added R27: 4.7k, Resistor_SMD:R_1206_3216Metric, B.Cu at (135.4, 94.3)
- added R28: 4.7k, Resistor_SMD:R_1206_3216Metric, B.Cu at (135.4, 90.7)
- added U11: PCA9306, Package_SO:SSOP-8_2.95x2.8mm_P0.65mm, B.Cu at (129.5, 92.2)
- C13, C14, C15, C17, C18, C27, C33, C35, C37, C38, C45, C46, C47, C48, C49, R21, R22, R23, U8: moved to B.Cu
- C7, C8, U4: moved to F.Cu
- D1, D2, D3, D4, D5, D6: footprint LED_SMD:LED_0805_2012Metric_Castellated -> LED_SMD:LED_0805_2012Metric_Pad1.15x1.40mm_HandSolder
- J1: value MiniPCIe LTE Modem -> Bus_PCI_Express_Mini
- MINI PCI-E CLIP: renamed from REF**
- Y2, Y3: footprint Crystal:Crystal_SMD_2016-4Pin_2.0x1.6mm -> Crystal:Crystal_SMD_HC49-SD
- moved R16 123.2 mm to (90.1, 143.1)
- moved C36 118.2 mm to (112.2, 137.9), turned to 270 degrees
- moved C34 113.9 mm to (121.7, 141.6), turned to 270 degrees
- moved C38 113.5 mm to (117.8, 139.5), turned to 90 degrees
- moved R24 113.2 mm to (114.3, 143.0), turned to 90 degrees
- moved C23 112.4 mm to (120.8, 144.8), turned to 180 degrees
- moved JP3 110.4 mm to (96.8, 143.1), turned to 180 degrees
- moved U5 109.3 mm to (106.7, 143.8), turned to 180 degrees
- moved C37 108.6 mm to (115.5, 134.6), turned to 180 degrees
- moved D3 106.8 mm to (137.8, 135.9), turned to 180 degrees
- moved JP1 106.7 mm to (116.2, 132.0)
- moved Y2 104.7 mm to (132.2, 143.7)
- moved C35 104.6 mm to (121.7, 141.6), turned to 270 degrees
- moved R15 103.0 mm to (117.2, 129.7), turned to 180 degrees
- moved Y3 100.4 mm to (103.7, 137.1), turned to 0 degrees
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Connections:
- C36 pad 2: +5V -> /USB2CAN_TRA/BOARD_5V
- C38 pad 1: +5V -> /USB2CAN_TRA/BOARD_5V
- C53 pad 1: +5V -> /USB2CAN_IMP/BOARD_5V
- C54 pad 2: +5V -> /USB2CAN_IMP/BOARD_5V
- J10 pad 1: Net-(J10-Pad1) -> GNDREF
- J10 pad 2: Net-(J10-Pad2) -> GNDREF
- J10 pad 3: Net-(J10-Pad3) -> GNDREF
- J10 pad 5: Net-(J10-Pad5) -> GNDREF
- J10 pad 7: Net-(J10-Pad7) -> GNDREF
- J5 pad 1: Net-(J5-Pad1) -> GNDREF
- J5 pad 3: Net-(J5-Pad1) -> GNDREF
- J5 pad 5: Net-(J5-Pad1) -> GNDREF
- J5 pad 7: Net-(J5-Pad1) -> GNDREF
- J6 pad 18: Net-(J6-Pad18) -> /Lattepanda/BOARD_SCL
- J6 pad 20: Net-(J6-Pad20) -> /Lattepanda/BOARD_SDA
- J6 pad 22: Net-(J6-Pad22) -> /Lattepanda/BOARD_1V8
- J7 pad 10: +5V -> Net-(J7-Pad10)
- J7 pad 4: +3V3 -> Net-(J7-Pad4)
- J7 pad 6: +3V3 -> Net-(J7-Pad4)
- J7 pad 8: +5V -> Net-(J7-Pad10)
- R21 pad 2: Net-(J6-Pad18) -> Net-(R21-Pad2)
- R22 pad 2: Net-(J6-Pad20) -> Net-(R22-Pad2)
- U10 pad 7: +5V -> /USB2CAN_IMP/BOARD_5V
- U2 pad 5: /USB_HUB/PRT_PWR_2 -> /USB2CAN_TRA/BOARD_5V
- U3 pad 8: /USB_HUB/PRT_PWR_3 -> /USB2CAN_IMP/BOARD_5V
- U5 pad 3: +5V -> /USB2CAN_TRA/BOARD_5V
- U7 pad 3: +5V -> /USB2CAN_IMP/BOARD_5V
- U8 pad 18: Net-(J6-Pad18) -> Net-(R21-Pad2)
- U8 pad 19: Net-(J6-Pad20) -> Net-(R22-Pad2)
- U9 pad 2: Net-(U9-Pad2) -> GNDREF
- U9 pad 7: +5V -> /USB2CAN_TRA/BOARD_5V
Routing:
- net GNDREF: track 128.9 -> 449.0 mm, vias 46 -> 73
- net Net-(R22-Pad2): track 0.00 -> 111.7 mm
- net +3V3: track 106.2 -> 216.1 mm, vias 17 -> 26
- net Net-(R21-Pad2): track 0.00 -> 96.2 mm
- net /USB2CAN_TRA/BOARD_5V: track 0.00 -> 55.3 mm, vias 0 -> 2
- net /USB2CAN_TRA/USB_DM: track 2.65 -> 54.1 mm
- net /USB_HEADERS/BOARD_5V: track 0.00 -> 48.3 mm, vias 0 -> 1
- net /USB2CAN_TRA/USB_DP: track 2.65 -> 50.2 mm
- net /USB2CAN_TRA/CAN_H: track 0.00 -> 45.2 mm
- net /USB2CAN_TRA/CAN_L: track 0.00 -> 44.2 mm
- net /USB2CAN_IMP/BOARD_5V: track 0.00 -> 41.8 mm, vias 0 -> 2
- net Net-(J7-Pad4): track 0.00 -> 41.2 mm
- net Net-(J13-Pad9): track 0.00 -> 38.3 mm
- net Net-(J13-Pad7): track 0.00 -> 36.8 mm
- net /USB_HEADERS/USB_DM: track 2.66 -> 37.0 mm
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- added copper zone on In1.Cu, net +3V3
- added copper zone on In1.Cu, net +5V
- added copper zone on In2.Cu, net GNDREF
Other:
- rule trace_min: 0.0889 -> 0.088

Commit message: Changed footprints for CAN connectors and replaced 3D models for headers
Parts:
- J14: renamed from MINI PCI-E CLIP
- J3, J4: footprint TerminalBlock_Phoenix:TerminalBlock_Phoenix_MKDS-1,5-3-5.08_1x03_P5.08mm_Horizontal -> TerminalBlock_Phoenix:TerminalBlock_Phoenix_PT-1,5-3-3.5-H_1x03_P3.50mm_Horizontal
- moved C19 20.5 mm to (164.0, 119.6), turned to 90 degrees
- moved C22 12.0 mm to (152.5, 138.2), turned to 180 degrees
- moved C21 2.24 mm to (146.9, 128.0), turned to 0 degrees
- moved R10 1.18 mm to (156.5, 123.7), turned to 180 degrees
- moved C20 0.58 mm to (148.4, 132.8)
- moved J2 0.30 mm to (158.2, 131.2), turned to 270 degrees
Routing:
- net Net-(C20-Pad1): track 25.2 -> 10.0 mm
- net GNDREF: track 449.0 -> 460.1 mm, vias 73 -> 71
- net Net-(C21-Pad1): track 23.7 -> 17.6 mm, vias 0 -> 2
- net Net-(J1-Pad16): track 32.1 -> 27.2 mm
- net Net-(C19-Pad1): track 37.1 -> 34.9 mm, vias 1 -> 2
- net Net-(C22-Pad1): track 21.5 -> 20.7 mm
- net /USB2CAN_IMP/CAN_L: track 26.6 -> 27.3 mm
Other:
- board text added: "CAN 1"
- board text added: "CAN 2"
- board text added: "LED PANEL OUT"
